Commit message: add files

File: turtlebot3_simulations/robot_gazebo/urdf/pav_s00/pav_s00.xacro (robot description, xacro)
@@ -159,6 +159,7 @@
     <axis xyz="0 0 1" />
     <limit lower="-0.5" upper="0.5" effort="5" velocity="1000" />
-  </joint>
-  <xacro:steering_hinge_transmission name="left_front_steer_hinge_link" />
+    <dynamics damping="0.1" friction="0.0"/>
+  </joint>
+  <!-- <xacro:steering_hinge_transmission name="left_front_steer_hinge_link" /> -->
   <link name="right_front_steer_hinge_link">
     <inertial>
@@ -199,6 +200,7 @@
     <axis xyz="0 0 1" />
     <limit lower="-0.5" upper="0.5" effort="5" velocity="1000" />
-  </joint>
-  <xacro:steering_hinge_transmission name="right_front_steer_hinge_link" />
+    <dynamics damping="0.1" friction="0.0"/>
+  </joint>
+  <!-- <xacro:steering_hinge_transmission name="right_front_steer_hinge_link" /> -->
   <link name="right_front_wheel_link">
     <inertial>
@@ -234,7 +236,7 @@
     <axis xyz="0 1 0" />
     <limit effort="10" velocity="1000" />
-    <dynamics damping="0.0" friction="${rotation_fiction}"/>
-  </joint>
-  <xacro:wheel_transmission name="right_front_wheel_link" />
+    <dynamics damping="0.1" friction="${rotation_fiction}"/>
+  </joint>
+  <!-- <xacro:wheel_transmission name="right_front_wheel_link" /> -->
   <link name="left_front_wheel_link">
     <inertial>
@@ -269,8 +271,8 @@
     <origin xyz="0 0.025 0" rpy="0 0 0" />
     <axis xyz="0 1 0" />
-    <!-- <limit effort="10" velocity="1000" />
-    <dynamics damping="0.0" friction="${rotation_fiction}"/> -->
-  </joint>
-  <xacro:wheel_transmission name="left_front_wheel_link" />
+    <limit effort="10" velocity="1000" />
+    <dynamics damping="0.1" friction="${rotation_fiction}"/>
+  </joint>
+  <!-- <xacro:wheel_transmission name="left_front_wheel_link" /> -->
   <link name="camera">
     <inertial>
